File: schematic/AC.sch (EAGLE design)
At the start: 37 parts, among them IC1 MEGA88/168/328-PU, IC3 78L33, Q1 32.768kHz, T1 BTA16-600, T2 BTA16-600, X1 MINI-USB, X2 230V IN, X3 L1 OUT, X4 L2 OUT

Commit message: Add files via upload
Parts:
- removed C5, C6: 10n 400V, resistor:C-EU102-043X133
- removed R11: 4k7, resistor:R-EU_0204/7
- R1: value 10K -> 10k
- R5: value 120K 1W -> 120k 1W
- R6, R7: value 1K 1W -> 390
- R8: value 39 1W -> 10k
- R9: value 39 1W -> 4k7; device resistor:R-EU_0207/10 -> resistor:R-EU_0204/7
- T1, T2: value BTA16-600 -> BTA16-600CW
Connections:
- removed net N$31: C5.1, R8.2
- removed net N$34: C6.1, R9.2
- removed net N$5: R5.1, R6.2, R7.2, R8.1, R9.1, T1.A2, T2.A2, X2-1.1
- new net N$1: OK1.AC2, R5.2
- net +3V3: now also IC1.AVCC, R8.1, R9.2; no longer R11.2
- net GND: now also JP3.3; no longer IC1.AVCC, JP3.2
- net N$11: now also R8.2
- net N$27: no longer C6.2
- net N$28: now also JP3.2, R9.1; no longer JP3.3, R10.1
- net N$35: no longer C5.2
- net N$36: now also R10.1; no longer R11.1
- net N$6: now also R6.2, R7.2, T1.A2, T2.A2, X2-1.1; no longer R5.2
- net N$7: now also R5.1; no longer OK1.AC2
Other:
- moved on the sheet: R10, R5, R8, R9, T1, T2, X2-1, X2-2, X3-1, X3-2, X4-1, X4-2

Commit message: Add files via upload
Parts:
- added R11, R12: 4k7, resistor:R-EU_0204/7
- IC1: value MEGA88/168/328-PU -> MEGA168/328-PU
- JP2: value RS232 -> I2C; device pinhead:PINHD-1X3 -> pinhead:PINHD-1X4
Connections:
- net +3V3: now also JP2.1, R11.2, R12.2
- net N$15: now also JP2.2, R11.1; no longer JP2.1
- net N$16: now also JP2.4, R12.1; no longer JP2.2
Other:
- note added: "SCL GND SDA VCC"
- note added: "VCC SDA GND SCL"
- moved on the sheet: JP3, R2, R5, S1, S2, S3, S4, U$1
